File: boards/u6502-sbc/u6502-sbc.kicad_sch (KiCad schematic)
At the start: 54 parts, among them J1 HDR_USR_PORT, J2 HDR_USR_PORT, J3 HDR_USR_PORT, J4 HDR_USR_PORT, J5 HDR_IRQ, J6 HDR_FTDI, J7 HDR_RS232, J8 KLDX-0202-BC, J9 HDR_CPU_BUS, SW1 SW_RST, SW2 SW_SPDT, U1 W65C02SxPL, U10 DS1813-5+, U2 AS7C256B-15PIN, U3 28C256, U4 W65C22SxPL, U5 W65C51NxP, U6 74HC00, U7 74HC21, U8 W65C22SxPL, U9 NCP1117IDT50T4G, X1 1MHz

Commit message: Initial layout and routing wip
Parts:
- removed RN2: 3k3, Resistor_THT:R_Array_SIP5, symbol Device:R_Network04
- added C20, C21, C23: 100n, Capacitor_THT:C_Rect_L4.0mm_W2.5mm_P2.50mm, symbol Device:C_Small
- added D1: LED_PWR, LED_THT:LED_D3.0mm, symbol Device:LED_Small
- added D2: 1N5819, Diode_THT:D_DO-41_SOD81_P7.62mm_Horizontal, symbol Device:D_Schottky
- added R1: 1k, Resistor_THT:R_Axial_DIN0204_L3.6mm_D1.6mm_P5.08mm_Horizontal, symbol Device:R_Small
- added X2: 1.8432 MHz, Oscillator:Oscillator_DIP-8, symbol Oscillator:CXO_DIP8
- C1, C10, C11, C12, C13, C14, C15, C16, C19, C2, C22, C3, C4, C5, C6, C7, C8, C9: footprint (none) -> Capacitor_THT:C_Rect_L4.0mm_W2.5mm_P2.50mm; Mfr (none) -> Vishay; Mfr Part (none) -> K104K15X7RF5TL2; Mouser Part (none) -> 594-K104K15X7RF5TL2
- C17: footprint Capacitor_Tantalum_SMD:CP_EIA-3528-21_Kemet-B_Pad1.50x2.35mm_HandSolder -> Capacitor_THT:CP_Radial_D8.0mm_P3.50mm; Mfr KYOCERA AVX -> KEMET; Mfr Part TAJB106M020RNJ -> ESL106M200AG9AA; Mouser Part (none) -> 80-ESL106M200AG9AA
- C18: value 10u -> 4u7; footprint Capacitor_Tantalum_SMD:CP_EIA-3528-21_Kemet-B_Pad1.50x2.35mm_HandSolder -> Capacitor_THT:CP_Radial_D5.0mm_P2.00mm; Mfr KYOCERA AVX -> Panasonic; Mfr Part TAJB106M020RNJ -> EEU-FR1H4R7B; Mouser Part (none) -> 667-EEU-FR1H4R7B
- F1: footprint Fuse:Fuse_1812_4532Metric_Pad1.30x3.40mm_HandSolder -> Fuse:Fuse_BelFuse_0ZRE0075FF_L11.5mm_W4.8mm; Mfr Eaton -> Bel Fuse; Mfr Part PTS181233V075 -> 0ZRG0075FF1E; Mouser Part (none) -> 530-0ZRG0075FF1E
- J1, J2, J3, J4: symbol Connector_Generic:Conn_02x07_Counter_Clockwise -> Connector_Generic:Conn_02x07_Odd_Even
- J5: footprint (none) -> Connector_PinHeader_2.54mm:PinHeader_2x04_P2.54mm_Vertical; symbol Connector_Generic:Conn_02x04_Counter_Clockwise -> Connector_Generic:Conn_02x04_Odd_Even
- J8: Mouser Part (none) -> 806-KLDX-0202-BC
- RN1: footprint Resistor_THT:R_Array_SIP5 -> Resistor_THT:R_Array_SIP7; symbol Device:R_Network04 -> Device:R_Network06; Mfr Part 4605X-101-332LF -> (none)
- SW2: Mouser Part (none) -> 633-GW12RCV
- U10: Mfr (none) -> Analog Devices; Mouser Part (none) -> 700-DS1813-5T&R
- U3: footprint Package_DIP:DIP-28_W15.24mm_Socket -> Mouser:Aries 28-526-10; Mfr (none) -> Aries Electronics; Mfr Part (none) -> 28-526-10; Mouser Part (none) -> 535-28-526-10
- U6: Mfr (none) -> Texas Instruments; Mfr Part (none) -> SN74HC00AN; Mouser Part (none) -> 595-SN74HC00AN
- U7: Mfr (none) -> Texas Instruments; Mfr Part (none) -> SN74HC21N; Mouser Part (none) -> 595-SN74HC21N
- U9: value NCP1117IDT50T4G -> L7805CV; footprint Package_TO_SOT_SMD:TO-252-2 -> Package_TO_SOT_THT:TO-220-3_Horizontal_TabDown; symbol Regulator_Linear:NCP1117-5.0_TO252 -> Regulator_Linear:LM7815_TO220; Mfr Onsemi -> STMicroelectronics; Mfr Part https://www.mouser.com/datasheet/2/308/NCP1117_D-2307187.pdf -> L7805CV; Mouser Part (none) -> 511-L7805CV
Connections:
- net ~{RST} is gone; now on net ~{RES}: SW1.1, U10.1 (~{RST})
- net BE: now also RN1.7 (R6), U1.40 (BE)
- net CA1: now also J1.11 (Pin_11); no longer J1.6 (Pin_6)
- net CA2: now also J1.12 (Pin_12); no longer J1.9 (Pin_9)
- net CB1: now also J2.11 (Pin_11); no longer J2.6 (Pin_6)
- net CB2: now also J2.12 (Pin_12); no longer J2.9 (Pin_9)
- net CC1: now also J3.11 (Pin_11); no longer J3.6 (Pin_6)
- net CC2: now also J3.12 (Pin_12); no longer J3.9 (Pin_9)
- net CD1: now also J4.11 (Pin_11); no longer J4.6 (Pin_6)
- net CD2: now also J4.12 (Pin_12); no longer J4.9 (Pin_9)
- net GND: now also J1.13 (Pin_13), J1.2 (Pin_2), J2.13 (Pin_13), J2.2 (Pin_2), J3.13 (Pin_13), J3.2 (Pin_2), J4.13 (Pin_13), J4.2 (Pin_2), U9.2 (GND), C20.1, C21.2, C23.2, D1.1 (K), X2.4 (GND); no longer J1.14 (Pin_14), J1.7 (Pin_7), J2.14 (Pin_14), J2.7 (Pin_7), J3.14 (Pin_14), J3.7 (Pin_7), J4.14 (Pin_14), J4.7 (Pin_7), U9.1 (GND)
- net IO_~{CS}: now also U8.25 (~{CS2})
- net IRQ0r: now also J5.2 (Pin_2); no longer J5.8 (Pin_8)
- net IRQ1r: now also J5.4 (Pin_4); no longer J5.7 (Pin_7)
- net IRQ3r: now also J5.8 (Pin_8); no longer J5.5 (Pin_5)
- net PA0: now also J1.3 (Pin_3); no longer J1.2 (Pin_2)
- net PA1: now also J1.5 (Pin_5); no longer J1.3 (Pin_3)
- net PA2: now also J1.7 (Pin_7); no longer J1.4 (Pin_4)
- net PA3: now also J1.9 (Pin_9); no longer J1.5 (Pin_5)
- net PA5: now also J1.8 (Pin_8); no longer J1.11 (Pin_11)
- net PA6: now also J1.6 (Pin_6); no longer J1.12 (Pin_12)
- net PA7: now also J1.4 (Pin_4); no longer J1.13 (Pin_13)
- net PB0: now also J2.3 (Pin_3); no longer J2.2 (Pin_2)
- net PB1: now also J2.5 (Pin_5); no longer J2.3 (Pin_3)
- net PB2: now also J2.7 (Pin_7); no longer J2.4 (Pin_4)
- net PB3: now also J2.9 (Pin_9); no longer J2.5 (Pin_5)
- net PB5: now also J2.8 (Pin_8); no longer J2.11 (Pin_11)
- net PB6: now also J2.6 (Pin_6); no longer J2.12 (Pin_12)
- net PB7: now also J2.4 (Pin_4); no longer J2.13 (Pin_13)
- net PC0: now also J3.3 (Pin_3); no longer J3.2 (Pin_2)
- net PC1: now also J3.5 (Pin_5); no longer J3.3 (Pin_3)
- net PC2: now also J3.7 (Pin_7); no longer J3.4 (Pin_4)
- net PC3: now also J3.9 (Pin_9); no longer J3.5 (Pin_5)
- net PC5: now also J3.8 (Pin_8); no longer J3.11 (Pin_11)
- net PC6: now also J3.6 (Pin_6); no longer J3.12 (Pin_12)
- net PC7: now also J3.4 (Pin_4); no longer J3.13 (Pin_13)
- net PD0: now also J4.3 (Pin_3); no longer J4.2 (Pin_2)
- net PD1: now also J4.5 (Pin_5); no longer J4.3 (Pin_3)
- net PD2: now also J4.7 (Pin_7); no longer J4.4 (Pin_4)
- net PD3: now also J4.9 (Pin_9); no longer J4.5 (Pin_5)
- net PD5: now also J4.8 (Pin_8); no longer J4.11 (Pin_11)
- net PD6: now also J4.6 (Pin_6); no longer J4.12 (Pin_12)
- net PD7: now also J4.4 (Pin_4); no longer J4.13 (Pin_13)
- net RDY: now also RN1.6 (R5), U1.3 (RDY)
- net SYNC: now also U1.8 (SYNC)
- net VCC: now also J1.14 (Pin_14), J2.14 (Pin_14), J3.14 (Pin_14), J4.14 (Pin_14), U9.3 (VO), C20.2, C21.1, C23.1, D2.2 (A), R1.1, X2.8 (Vcc); no longer J1.8 (Pin_8), J2.8 (Pin_8), J3.8 (Pin_8), J4.8 (Pin_8), U9.2 (VO)
- net VDC: now also U9.1 (VI), D2.1 (K); no longer U9.3 (VI)
- net ~{IRQ1}: now also J5.3 (Pin_3); no longer J5.2 (Pin_2)
- net ~{IRQ2}: now also J5.5 (Pin_5); no longer J5.3 (Pin_3)
- net ~{IRQ3}: now also J5.7 (Pin_7); no longer J5.4 (Pin_4)
- net ftdi_vcc: now reaches J6.4 (Pin_4), JP1.2 (B)
- net ACIA_XTAL: now reaches U5.6 (XTAL1)
- net ACIA_XTAL: now also X2.5 (OUT)
- new net pwr_led_r: D1.2 (A), R1.2
- no-connect marks 10 -> 19
Other:
- note added: "DC Power Regulation"
- moved on the sheet: C17, C18, F1, J8, SW2, U9

Commit message: Board rev 0 ordered
Parts:
- removed TH1, TH2, TH3: ToolingHole, JLCPCB_SMT:ToolingHole, symbol JLCPCB_SMT:ToolingHole
- added HS1: Heatsink, symbol Mechanical:Heatsink
Other:
- note added: "Address Decode Logic"
- note added: "Address Map"
- note added: "CPU Bus Debug Header"
- note added: "Interrupt Logic"
- note added: "RAM: $0000 - $3FFF ACIA: $4400 - $4403 VIA2: $5000 - $500F VIA1: $6000 - $600F ROM: $8000 - $FFFF"
- note added: "Reset Circuit"
- note added: "System Clock"
- note added: "TTL Serial UART (ACIA)"
- note added: "User Ports (VIAs 1 & 2)"
- note removed: "Tooling Holes"
- moved on the sheet: C10, C11, C12, C13, C14, C15, C19, C2, C20, C22, C5, C6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
